Commit message: [Iter#2 rerobDesgn-1] Modifying Arm Design. Now 6 DOF

File: robotarm_description/urdf/robotinitial.urdf (robot description, URDF)
Before this commit: robot simpleArm, 4 links, 3 joints
Joints:
- joint first_to_second_link: origin xyz=0 0.1 0 rpy=0 1.57 0 -> xyz=0 0.15 0 rpy=0 1.57 0
