Commit message: [Iter#2 simset-1] Add Gazebo Elements to the robot model

File: robotarm_description/urdf/robotArm.xacro (robot description, xacro)
@@ -4,4 +4,6 @@
 -->
 <robot name="six_dof_arm" xmlns:xacro="http://www.ros.org/wiki/xacro">
+<!-- Include Gazebo Properties-->
+<xacro:include filename="$(find robotarm_description)/urdf/robotArm.gazebo.xacro" />
 <!-- Include materials -->
     <material name="Blue">
@@ -56,4 +58,11 @@
       <material name="White"/>
     </visual>
+  <collision>
+      <origin xyz="0 0 0" rpy="0 0 0" /> <!-- rotate PI/2 -->
+      <geometry>
+         <box size="${base_link_width} ${base_link_depth} ${base_link_height}" />
+      </geometry>
+  </collision>
+<xacro:inertial_matrix mass="1"/>
 </link>
 <!-- BASE LINK -->
@@ -66,9 +75,16 @@
     <material name="White"/>
     </visual>
+  <collision>
+      <origin xyz="0 0 0" rpy="0 0 0" /> <!-- rotate PI/2 -->
+      <geometry>
+         <cylinder radius="0.04" length="${base_link2_height}"/>
+      </geometry>
+  </collision>
+  <xacro:inertial_matrix mass="1"/>
 </link>
 <joint name="shoulder_pan_joint" type="revolute">
     <parent link="base_link_2"/>
     <child link="shoulder_pan_link"/>
-    <origin xyz="0 0 0.02" rpy="0 0 -1.573" />
+    <origin xyz="0 0 0.02" rpy="0 0 -${M_PI/2}" />
     <axis xyz="0 0 1" />
     <limit effort="300" velocity="1" lower="-2.61799387799" upper="1.98394848567"/>
@@ -84,9 +100,16 @@
       <material name="Red"/>
     </visual>
+    <collision>
+      <origin xyz="0 0 0" rpy="0 0 0" />
+      <geometry>
+            <cylinder radius="${shoulder_pan_width}" length="${shoulder_pan_len}"/>
+      </geometry>
+    </collision>
+<xacro:inertial_matrix mass="1"/>
 </link>
   <joint name="shoulder_pitch_joint" type="revolute">
     <parent link="shoulder_pan_link"/>
     <child link="shoulder_pitch_link"/>
-    <origin xyz="-0.041 0.0021 0.0" rpy="-1.573 0 1.573" />
+    <origin xyz="-0.041 0.0021 0.0" rpy="-${M_PI/2} 0 ${M_PI/2}" />
     <axis xyz="1 0 0" />
     <limit effort="300" velocity="1" lower="-1.19962513147" upper="1.89994105047" />
@@ -96,5 +119,5 @@
   <link name="shoulder_pitch_link" >
     <visual>
-      <origin xyz="-0.002 0 0.04" rpy="0 1.573 0" />
+      <origin xyz="-0.002 0 0.04" rpy="0 ${M_PI/2} 0" />
       <geometry>
            <box size="${shoulder_pitch_len} ${shoulder_pitch_width} ${shoulder_pitch_height}" />
@@ -102,9 +125,16 @@
     <material name="Blue"/>
     </visual>
+    <collision>
+      <origin xyz="-0.002 0 0.04" rpy="0 ${M_PI/2} 0" />
+      <geometry>
+           <box size="${shoulder_pitch_len} ${shoulder_pitch_width} ${shoulder_pitch_height}" />
+      </geometry>
+    </collision>
+    <xacro:inertial_matrix mass="1"/>
 </link>
  <joint name="elbow_roll_joint" type="revolute">
     <parent link="shoulder_pitch_link"/>
     <child link="elbow_roll_link"/>
-    <origin xyz="-0.002 0 0.1206" rpy="3.146 1.573 0" />
+    <origin xyz="-0.002 0 0.1206" rpy="${M_PI} ${M_PI/2} 0" />
     <axis xyz="-1 0 0" />
     <limit effort="300" velocity="1" lower="-2.61799387799" upper="0.705631162427" />
@@ -114,5 +144,5 @@
   <link name="elbow_roll_link" >
     <visual>
-      <origin xyz="-0.015 0.0 -0.0" rpy="0 1.573 0" />
+      <origin xyz="-0.015 0.0 -0.0" rpy="0 ${M_PI/2} 0" />
       <geometry>
             <cylinder radius= "${elbow_roll_width}" length="${elbow_roll_len}"/>
@@ -120,9 +150,16 @@
    <material name="Red"/>
     </visual>
+    <collision>
+      <origin xyz="-0.015 0.0 -0.0" rpy="0 ${M_PI/2} 0" />
+      <geometry>
+            <cylinder radius="${elbow_roll_width}" length="${elbow_roll_len}"/>
+      </geometry>
+    </collision>
+    <xacro:inertial_matrix mass="1"/>
 </link>
 <joint name="elbow_pitch_joint" type="revolute">
     <parent link="elbow_roll_link"/>
     <child link="elbow_pitch_link"/>
-    <origin xyz="-0.035 0 0.0" rpy="0.055 1.573 0" />
+    <origin xyz="-0.035 0 0.0" rpy="0.055 ${M_PI/2} 0" />
     <axis xyz="1 0 0" />
     <limit effort="300" velocity="1" lower="-1.5953400194" upper="1.93281579274" />
@@ -132,5 +169,5 @@
   <link name="elbow_pitch_link" >
     <visual>
-      <origin xyz="0 0 -0.12" rpy="0 1.573 0" />
+      <origin xyz="0 0 -0.12" rpy="0 ${M_PI/2} 0" />
       <geometry>
        <box size="${elbow_pitch_len} ${elbow_pitch_width} ${elbow_pitch_height}" />
@@ -138,9 +175,16 @@
     <material name="Blue"/>
     </visual>
+    <collision>
+      <origin xyz="0 0 -0.12" rpy="0 ${M_PI/2} 0" />
+      <geometry>
+       <box size="${elbow_pitch_len} ${elbow_pitch_width} ${elbow_pitch_height}" />
+      </geometry>
+    </collision>
+    <xacro:inertial_matrix mass="1"/>
 </link>
 <joint name="wrist_roll_joint" type="revolute">
     <parent link="elbow_pitch_link"/>
     <child link="wrist_roll_link"/>
-    <origin xyz="0.0 0.0081 -.248" rpy="0 1.573 3.146" />
+    <origin xyz="0.0 0.0081 -.248" rpy="0 ${M_PI/2} ${M_PI}" />
     <axis xyz="1 0 0" />
     <limit effort="300" velocity="1" lower="-2.61799387799" upper="2.6128806087" />
@@ -149,5 +193,5 @@
 <link name="wrist_roll_link" >
     <visual>
-      <origin xyz="0 0 0" rpy="0 1.573 0" />
+      <origin xyz="0 0 0" rpy="0 ${M_PI/2} 0" />
       <geometry>
            <cylinder radius="${wrist_roll_width}" length="${wrist_roll_len}"/>
@@ -155,9 +199,16 @@
     <material name="Red"/>
     </visual>
+  <collision>
+      <origin xyz="0 0 0" rpy="0 ${M_PI/2} 0" />
+      <geometry>
+           <cylinder radius="${wrist_roll_width}" length="${wrist_roll_len}"/>
+      </geometry>
+  </collision>
+  <xacro:inertial_matrix mass="1"/>
 </link>
 <joint name="wrist_pitch_joint" type="revolute">
     <parent link="wrist_roll_link"/>
     <child link="wrist_pitch_link"/>
-    <origin xyz="0.0 0.0 0.0001" rpy="0 1.573 0" />
+    <origin xyz="0.0 0.0 0.0001" rpy="0 ${M_PI/2} 0" />
     <axis xyz="1 0 0" />
     <limit effort="300" velocity="1" lower="-1.5953400194" upper="1.98394848567" />
@@ -167,5 +218,5 @@
   <link name="wrist_pitch_link">
     <visual>
-      <origin xyz="0 0 0.04" rpy="0 1.573 0" />
+      <origin xyz="0 0 0.04" rpy="0 ${M_PI/2} 0" />
       <geometry>
            <box size="${wrist_pitch_len} ${wrist_pitch_width} ${wrist_pitch_height}" />
@@ -173,4 +224,18 @@
     <material name="Blue"/>
     </visual>
-</link>
+    <collision>
+      <origin xyz="0 0 0.04 " rpy="0 ${M_PI/2} 0" />
+      <geometry>
+          <box size="${wrist_pitch_len} ${wrist_pitch_width} ${wrist_pitch_height}" />
+      </geometry>
+    </collision>
+    <xacro:inertial_matrix mass="1"/>
+</link>
+<!-- Initiate Transmission Tags for Each joint-->
+   <xacro:transmission_block joint_name="shoulder_pan_joint"/>
+   <xacro:transmission_block joint_name="shoulder_pitch_joint"/>
+   <xacro:transmission_block joint_name="elbow_roll_joint"/>
+   <xacro:transmission_block joint_name="elbow_pitch_joint"/>
+   <xacro:transmission_block joint_name="wrist_roll_joint"/>
+   <xacro:transmission_block joint_name="wrist_pitch_joint"/>
 </robot>

Commit message: [Iter#2 simset-3] Initial Attempts to setup camera Table and Object. Needs More Work

File: robotarm_description/urdf/robotArm.xacro (robot description, xacro)
@@ -21,5 +21,5 @@
   <property name="base_link_width" value="0.5" />
   <property name="base_link_depth" value="0.06" />
-  <property name="base_link_height" value="0.6" />
+  <property name="base_link_height" value="1" />
   <property name="base_link2_height" value = "0.02" />
  <!-- Shoulder pan link properties -->
@@ -45,5 +45,5 @@
   <property name="wrist_pitch_height" value="0.04" />
   <joint name="bottom_joint2" type="fixed">
-    <origin xyz="0.15 0.07 0.15" rpy="0 0 0" />
+    <origin xyz="0.15 0.07 0.38" rpy="0 0 0" />
     <parent link="base_link"/>
     <child link="base_link_2"/>
@@ -110,5 +110,5 @@
     <parent link="base_link_2"/>
     <child link="shoulder_pan_link"/>
-    <origin xyz="0 0 0.02" rpy="0 0 -${M_PI/2}" />
+    <origin xyz="0 0 0.02" rpy="0 0 -${M_PI}" />
     <axis xyz="0 0 1" />
     <limit effort="300" velocity="1" lower="-2.61799387799" upper="1.98394848567"/>
@@ -185,6 +185,6 @@
     <parent link="elbow_roll_link"/>
     <child link="elbow_pitch_link"/>
-    <origin xyz="-0.035 0 0.0" rpy="0.055 ${M_PI/2} 0" />
-    <axis xyz="1 0 0" />
+    <origin xyz="-0.035 0 0.0" rpy="${-M_PI/2} 0 0"/> <!-- 0.055-->
+    <axis xyz="0 1 0" />
     <limit effort="300" velocity="1" lower="-1.5953400194" upper="1.93281579274" />
     <dynamics damping="50" friction="1"/>
@@ -256,4 +256,5 @@
     <xacro:inertial_matrix mass="1"/>
 </link>
+<xacro:include filename="$(find robotarm_description)/urdf/sensors/camera.urdf.xacro"/>
 <!-- Initiate Transmission Tags for Each joint-->
    <xacro:transmission_block joint_name="shoulder_pan_joint"/>

Commit message: [Iter#3 cvInt] Integration of openCV algorithm and ROS using cv_bridge

File: robotarm_description/urdf/robotArm.xacro (robot description, xacro)
@@ -72,5 +72,5 @@
   <link name="bottom_link">
     <visual>
-      <origin xyz=" 0 0 -${base_link_height/2}"  rpy="0 0 0"/>
+      <origin xyz=" 0 0 -${base_link_height/2 + 0.01}"  rpy="0 0 0"/>
       <geometry>
          <box size="0.2 0.2 0.02" />
@@ -79,10 +79,10 @@
     </visual>
     <collision>
-      <origin xyz=" 0 0 -0.04"  rpy="0 0 0"/>
+      <origin xyz=" 0 0 -${base_link_height/2 + 0.01}"  rpy="0 0 0"/>
       <geometry>
          <box size="0.2 0.2 0.02" />
       </geometry>
       </collision>>
-      <xacro:inertial_matrix mass="1000"/>
+      <xacro:inertial_matrix mass="10"/>
   </link>
   <gazebo reference="bottom_link">

Commit message: [Iter#3 simset-2] Minor change for better stability of robot

File: robotarm_description/urdf/robotArm.xacro (robot description, xacro)
@@ -74,14 +74,14 @@
       <origin xyz=" 0 0 -${base_link_height/2 + 0.01}"  rpy="0 0 0"/>
       <geometry>
+         <box size="0.5 0.2 0.02" />
+      </geometry>
+      <material name="Brown" />
+    </visual>
+    <!--collision>
+      <origin xyz=" 0 0 -${base_link_height/2 + 0.01}"  rpy="0 0 0"/>
+      <geometry>
          <box size="0.2 0.2 0.02" />
       </geometry>
-      <material name="Brown" />
-    </visual>
-    <collision>
-      <origin xyz=" 0 0 -${base_link_height/2 + 0.01}"  rpy="0 0 0"/>
-      <geometry>
-         <box size="0.2 0.2 0.02" />
-      </geometry>
-      </collision>>
+      </collision-->
       <xacro:inertial_matrix mass="90"/>
   </link>
