Commit message: [Iter#2 simset-2] Robot Arm Spawned in Gazebo

File: robotarm_description/urdf/robotArm.gazebo.xacro (robot description, xacro)
@@ -33,19 +33,25 @@
   <gazebo reference="shoulder_pan_link">
     <material>Gazebo/Red</material>
+    <turnGravityOff>true</turnGravityOff>
 </gazebo>
 <gazebo reference="shoulder_pitch_link">
     <material>Gazebo/Blue</material>
+    <turnGravityOff>true</turnGravityOff>
 </gazebo>
   <gazebo reference="elbow_roll_link">
     <material>Gazebo/Red</material>
+    <turnGravityOff>true</turnGravityOff>
 </gazebo>
  <gazebo reference="elbow_pitch_link">
     <material>Gazebo/Blue</material>
+    <turnGravityOff>true</turnGravityOff>
 </gazebo>
 <gazebo reference="wrist_roll_link">
     <material>Gazebo/Red</material>
+    <turnGravityOff>true</turnGravityOff>
 </gazebo>
   <gazebo reference="wrist_pitch_link">
     <material>GazeboBlue</material>
+    <turnGravityOff>true</turnGravityOff>
 </gazebo>
 <!-- ros_control plugin -->
@@ -53,5 +59,10 @@
     <plugin name="gazebo_ros_control" filename="libgazebo_ros_control.so">
       <robotNamespace>/robot_arm</robotNamespace>
+      <turnGravityOff>true</turnGravityOff>
     </plugin>
 </gazebo>
+ <gazebo reference="base_link">
+    <static>true</static>
+    <turnGravityOff>true</turnGravityOff>
+</gazebo>
 	</robot>

File: robotarm_description/urdf/robotArm.xacro (robot description, xacro)
@@ -21,5 +21,5 @@
   <property name="base_link_width" value="0.5" />
   <property name="base_link_depth" value="0.06" />
-  <property name="base_link_height" value="1" />
+  <property name="base_link_height" value="0.6" />
   <property name="base_link2_height" value = "0.02" />
  <!-- Shoulder pan link properties -->
@@ -45,8 +45,32 @@
   <property name="wrist_pitch_height" value="0.04" />
   <joint name="bottom_joint2" type="fixed">
-    <origin xyz="0.15 0.07 0.38" rpy="0 0 0" />
+    <origin xyz="0.15 0.07 0.15" rpy="0 0 0" />
     <parent link="base_link"/>
     <child link="base_link_2"/>
 </joint>
+<joint name="bottom_joint" type="fixed">
+    <origin xyz="0 0 0" rpy="0 0 0" />
+    <parent link="base_link"/>
+    <child link="bottom_link"/>
+  </joint>
+  <link name="bottom_link">
+    <visual>
+      <origin xyz=" 0 0 -${base_link_height/2}"  rpy="0 0 0"/>
+      <geometry>
+         <box size="0.5 0.5 0.02" />
+      </geometry>
+      <material name="Brown" />
+    </visual>
+    <collision>
+      <origin xyz=" 0 0 -0.04"  rpy="0 0 0"/>
+      <geometry>
+         <box size="1 1 0.02" />
+      </geometry>
+      </collision>>
+      <xacro:inertial_matrix mass="100"/>
+  </link>
+  <gazebo reference="bottom_link">
+    <material>Gazebo/White</material>
+</gazebo>
 <!-- BASE LINK -->
   <link name="base_link">

Commit message: [iter#2 simset-4] Siumlation Setup with Table, Object and Robot. Add World file

File: robotarm_description/urdf/robotArm.gazebo.xacro (robot description, xacro)
@@ -30,4 +30,5 @@
  <gazebo reference="base_link_2">
     <material>Gazebo/White</material>
+    <turnGravityOff>true</turnGravityOff>
 </gazebo>
   <gazebo reference="shoulder_pan_link">
@@ -64,5 +65,5 @@
  <gazebo reference="base_link">
     <static>true</static>
-    <turnGravityOff>true</turnGravityOff>
+    <!-- turnGravityOff>true</turnGravityOff!-->
 </gazebo>
 	</robot>

File: robotarm_description/urdf/sensors/camera.gazebo.xacro (robot description, xacro)
@@ -9,5 +9,5 @@
       <update_rate>30.0</update_rate>
       <camera name="head">
-        <horizontal_fov>.95</horizontal_fov>
+        <horizontal_fov>0.95</horizontal_fov>
         <!-- <horizontal_fov>0.95</horizontal_fov> -->
         <image>

File: robotarm_description/urdf/sensors/camera.urdf.xacro (robot description, xacro)
@@ -5,5 +5,5 @@
 <robot name="six_dof_arm" xmlns:xacro="http://www.ros.org/wiki/xacro">
 <joint name="camera_joint" type="fixed">
-    <origin xyz="0 0.5 1" rpy="${M_PI} 0 0"/>
+    <origin xyz="0 0.2 2" rpy="${M_PI} 0 0"/>
     <parent link="base_link"/>
     <child link="camera_link"/>

Commit message: [Iter#2 impl-1] Implementing stub classes for Object Recognition

File: robotarm_description/urdf/robotArm.gazebo.xacro (robot description, xacro)
@@ -23,11 +23,11 @@
 <!-- Material References of the Links for Gazebo-->
   <gazebo reference="bottom_link">
-    <material>Gazebo/White</material>
+    <material>Gazebo/Black</material>
 </gazebo>
  <gazebo reference="base_link">
-    <material>Gazebo/White</material>
+    <material>Gazebo/Black</material>
 </gazebo>
  <gazebo reference="base_link_2">
-    <material>Gazebo/White</material>
+    <material>Gazebo/Black</material>
     <turnGravityOff>true</turnGravityOff>
 </gazebo>
@@ -53,5 +53,5 @@
 </gazebo>
   <gazebo reference="wrist_pitch_link">
-    <material>GazeboBlue</material>
+    <material>Gazebo/Blue</material>
     <turnGravityOff>true</turnGravityOff>
 </gazebo>

File: robotarm_description/urdf/robotArm.xacro (robot description, xacro)
@@ -71,5 +71,5 @@
   </link>
   <gazebo reference="bottom_link">
-    <material>Gazebo/White</material>
+    <material>Gazebo/Black</material>
 </gazebo>
 <!-- BASE LINK -->

Commit message: [Iter-3 robDesgn-2 Adding the Gripper to the Robot

File: robotarm_description/urdf/robotArm.gazebo.xacro (robot description, xacro)
@@ -56,4 +56,16 @@
     <turnGravityOff>true</turnGravityOff>
 </gazebo>
+<gazebo reference="gripper_roll_link">
+    <material>Gazebo/Red</material>
+    <turnGravityOff>true</turnGravityOff>
+</gazebo>
+<gazebo reference="l_gripper_aft_link">
+    <material>Gazebo/White</material>
+    <turnGravityOff>true</turnGravityOff>
+</gazebo>
+<gazebo reference="r_gripper_aft_link">
+    <material>Gazebo/White</material>
+    <turnGravityOff>true</turnGravityOff>
+</gazebo>
 <!-- ros_control plugin -->
   <gazebo>
@@ -65,5 +77,9 @@
  <gazebo reference="base_link">
     <static>true</static>
-    <!-- turnGravityOff>true</turnGravityOff!-->
+    <turnGravityOff>true</turnGravityOff>
+</gazebo>
+ <gazebo reference="bottom_link">
+    <static>true</static>
+    <!-- turnGravityOff>true</turnGravityOff -->
 </gazebo>
 	</robot>

File: robotarm_description/urdf/robotArm.xacro (robot description, xacro)
@@ -44,4 +44,20 @@
   <property name="wrist_pitch_width" value="0.04" />
   <property name="wrist_pitch_height" value="0.04" />
+  <!--Gripper Parameters taken from https://github.com/qboticslabs/mastering_ros/blob/master/chapter_3_codes/mastering_ros_robot_description_pkg/urdf/seven_dof_arm.xacro -->
+<!-- Gripper roll link properties -->
+  <property name="gripper_roll_width" value="0.04" />
+  <property name="gripper_roll_len" value="0.02" />
+  <!-- Left gripper -->
+  <property name="left_gripper_len" value="0.08" />
+  <property name="left_gripper_width" value="0.01" />
+  <property name="left_gripper_height" value="0.01" />
+  <!-- Right gripper -->
+  <property name="right_gripper_len" value="0.08" />
+  <property name="right_gripper_width" value="0.01" />
+  <property name="right_gripper_height" value="0.01" />
+  <!-- Right gripper -->
+  <property name="grasp_frame_len" value="0.02" />
+  <property name="grasp_frame_width" value="0.02" />
+  <property name="grasp_frame_height" value="0.02" />
   <joint name="bottom_joint2" type="fixed">
     <origin xyz="0.15 0.07 0.38" rpy="0 0 0" />
@@ -68,5 +84,5 @@
       </geometry>
       </collision>>
-      <xacro:inertial_matrix mass="100"/>
+      <xacro:inertial_matrix mass="1000"/>
   </link>
   <gazebo reference="bottom_link">
@@ -88,5 +104,5 @@
       </geometry>
   </collision>
-<!-- xacro:inertial_matrix mass="1" -->
+ <xacro:inertial_matrix mass="1"/>
 </link>
 <!-- BASE LINK -->
@@ -112,5 +128,5 @@
     <origin xyz="0 0 0.02" rpy="0 0 -${M_PI}" />
     <axis xyz="0 0 1" />
-    <limit effort="300" velocity="1" lower="-2.61799387799" upper="1.98394848567"/>
+    <limit effort="300" velocity="1" lower="-0.05" upper="2.61799387799"/>
     <dynamics damping="50" friction="1"/>
 </joint>
@@ -162,5 +178,5 @@
     <origin xyz="-0.002 0 0.1206" rpy="${M_PI} ${M_PI/2} 0" />
     <axis xyz="-1 0 0" />
-    <limit effort="300" velocity="1" lower="-2.61799387799" upper="0.705631162427" />
+    <limit effort="300" velocity="1" lower="-0.705631162427" upper="2.61799387799" />
     <dynamics damping="50" friction="1"/>
 </joint>
@@ -235,5 +251,5 @@
     <child link="wrist_pitch_link"/>
     <origin xyz="0.0 0.0 0.0001" rpy="0 ${M_PI/2} 0" />
-    <axis xyz="1 0 0" />
+    <axis xyz="0 1 0" />
     <limit effort="300" velocity="1" lower="-1.5953400194" upper="1.98394848567" />
     <dynamics damping="50" friction="1"/>
@@ -256,4 +272,105 @@
     <xacro:inertial_matrix mass="1"/>
 </link>
+  <!-- Following Gripper Design is taken from https://github.com/qboticslabs/mastering_ros/blob/master/chapter_3_codes/mastering_ros_robot_description_pkg/urdf/seven_dof_arm.xacro-->
+  <joint name="gripper_roll_joint" type="revolute">
+    <parent link="wrist_pitch_link"/>
+    <child link="gripper_roll_link"/>
+    <origin xyz="0 0 0.080" rpy="${1.5*M_PI} -${.5*M_PI} 0" />
+    <axis xyz="1 0 0" />
+    <limit effort="300" velocity="1" lower="-2.61799387799" upper="2.6128806087" />
+    <dynamics damping="50" friction="1"/>
+</joint>
+<!-- GRIPPER ROLL LINK -->
+  <link name="gripper_roll_link">
+    <visual>
+      <origin xyz="0 0 0" rpy="0 ${M_PI/2} 0" />
+      <geometry>
+            <cylinder radius="${gripper_roll_width}" length="${gripper_roll_len}"/>
+      </geometry>
+      <material name="Red" />
+    </visual>
+    <collision>
+      <origin xyz="0 0 0" rpy="0 ${M_PI/2} 0" />
+      <geometry>
+            <cylinder radius="${gripper_roll_width}" length="${gripper_roll_len}"/>
+      </geometry>
+    </collision>
+  <xacro:inertial_matrix mass="1"/>
+  </link>
+  <gazebo reference="gripper_roll_link">
+    <material>Gazebo/Red</material>
+  </gazebo>
+  <joint name="finger_joint1" type="prismatic">
+    <parent link="gripper_roll_link"/>
+    <child link="gripper_finger_link1"/>
+    <origin xyz="0.0 0 0" />
+    <axis xyz="0 1 0" />
+      <limit effort="100" lower="0.03" upper="0" velocity="1.0"/>
+      <safety_controller k_position="20"
+                         k_velocity="20"
+                         soft_lower_limit="${-0.15 }"
+                         soft_upper_limit="${ 0.0 }"/>
+    <dynamics damping="50" friction="1"/>
+  </joint>
+<!-- ///////////////////////////////////////////////////////////////////////////////////////////////////////////////////// -->
+  <!-- LEFT GRIPPER AFT LINK -->
+  <link name="gripper_finger_link1">
+     <visual>
+      <origin xyz="0.04 -0.03 0"/>
+      <geometry>
+           <box size="${left_gripper_len} ${left_gripper_width} ${left_gripper_height}" />
+      </geometry>
+      <material name="White" />
+    </visual>
+  <xacro:inertial_matrix mass="1"/>
+  </link>
+  <gazebo reference="l_gripper_aft_link">
+    <material>Gazebo/White</material>
+  </gazebo>
+<!-- Joint between Wrist roll and finger 2 -->
+  <joint name="finger_joint2" type="prismatic">
+    <parent link="gripper_roll_link"/>
+    <child link="gripper_finger_link2"/>
+    <origin xyz="0.0 0 0" />
+    <axis xyz="0 1 0" />
+    <limit effort="1" lower="-0.03" upper="0" velocity="1.0"/>
+    <dynamics damping="50" friction="1"/>
+  </joint>
+<!-- ///////////////////////////////////////////////////////////////////////////////////////////////////////////////////// -->
+  <!-- RIGHT GRIPPER AFT LINK -->
+  <link name="gripper_finger_link2">
+    <visual>
+      <origin xyz="0.04 0.03 0"/>
+      <geometry>
+          <box size="${right_gripper_len} ${right_gripper_width} ${right_gripper_height}" />
+      </geometry>
+      <material name="White" />
+    </visual>
+  <xacro:inertial_matrix mass="1"/>
+  </link>
+  <gazebo reference="r_gripper_aft_link">
+    <material>Gazebo/White</material>
+  </gazebo>
+    <!-- Grasping frame -->
+    <link name="grasping_frame">
+      <inertial>
+        <origin xyz="0 0 0" rpy="0 0 0"/>
+        <mass value="0.0001"/>
+        <cuboid_inertia mass="0.0001" x="0.001" y="0.001" z="0.001"/>
+        <inertia  ixx="1.0" ixy="0.0"  ixz="0.0"  iyy="100.0"  iyz="0.0"  izz="1.0" />
+      </inertial>
+    <visual>
+      <origin xyz="0 0 0"/>
+      <geometry>
+          <box size="${grasp_frame_len} ${grasp_frame_width} ${grasp_frame_height}" />
+      </geometry>
+      <material name="White" />
+    </visual>
+    </link>
+    <joint name="grasping_frame_joint" type="fixed">
+      <parent link="gripper_roll_link"/>
+      <child link="grasping_frame"/>
+      <origin xyz="0.08 0 0" rpy="0 0 0"/>
+</joint>
 <xacro:include filename="$(find robotarm_description)/urdf/sensors/camera.urdf.xacro"/>
 <!-- Initiate Transmission Tags for Each joint-->
@@ -264,3 +381,6 @@
    <xacro:transmission_block joint_name="wrist_roll_joint"/>
    <xacro:transmission_block joint_name="wrist_pitch_joint"/>
+   <xacro:transmission_block joint_name="gripper_roll_joint"/>
+   <xacro:transmission_block joint_name="finger_joint1"/>
+   <xacro:transmission_block joint_name="finger_joint2"/>
 </robot>

Commit message: [iter#3 simset-1] Miscellaneous changes for obtaining a feasible simulation setup

File: robotarm_description/urdf/robotArm.gazebo.xacro (robot description, xacro)
@@ -27,4 +27,6 @@
  <gazebo reference="base_link">
     <material>Gazebo/Black</material>
+    <static>true</static>
+    <turnGravityOff>true</turnGravityOff>
 </gazebo>
  <gazebo reference="base_link_2">
@@ -68,14 +70,14 @@
     <turnGravityOff>true</turnGravityOff>
 </gazebo>
+<gazebo reference="camera_link">
+    <material>Gazebo/Black</material>
+    <turnGravityOff>true</turnGravityOff>
+</gazebo>
 <!-- ros_control plugin -->
-  <gazebo>
+<gazebo>
     <plugin name="gazebo_ros_control" filename="libgazebo_ros_control.so">
       <robotNamespace>/robot_arm</robotNamespace>
       <turnGravityOff>true</turnGravityOff>
     </plugin>
-</gazebo>
- <gazebo reference="base_link">
-    <static>true</static>
-    <turnGravityOff>true</turnGravityOff>
 </gazebo>
  <gazebo reference="bottom_link">

File: robotarm_description/urdf/robotArm.xacro (robot description, xacro)
@@ -61,5 +61,5 @@
   <property name="grasp_frame_height" value="0.02" />
   <joint name="bottom_joint2" type="fixed">
-    <origin xyz="0.15 0.07 0.38" rpy="0 0 0" />
+    <origin xyz="0.15 0.07 0.45" rpy="0 0 0" />
     <parent link="base_link"/>
     <child link="base_link_2"/>
@@ -74,5 +74,5 @@
       <origin xyz=" 0 0 -${base_link_height/2}"  rpy="0 0 0"/>
       <geometry>
-         <box size="0.5 0.5 0.02" />
+         <box size="0.2 0.2 0.02" />
       </geometry>
       <material name="Brown" />
@@ -81,5 +81,5 @@
       <origin xyz=" 0 0 -0.04"  rpy="0 0 0"/>
       <geometry>
-         <box size="1 1 0.02" />
+         <box size="0.2 0.2 0.02" />
       </geometry>
       </collision>>
@@ -104,5 +104,5 @@
       </geometry>
   </collision>
- <!-- xacro:inertial_matrix mass="1" -->
+ <!--xacro:inertial_matrix mass="1"-->
 </link>
 <!-- BASE LINK -->

File: robotarm_description/urdf/sensors/camera.urdf.xacro (robot description, xacro)
@@ -25,5 +25,5 @@
    </visual>
    <inertial>
-   <mass value="1e-5" />
+   <mass value="1e-6" />
    <origin xyz="0 0 0" rpy="0  0 0"/>
    <inertia ixx="1e-6" ixy="0" ixz="0" iyy="1e-6" iyz="0" izz="1e-6" />

Commit message: [Iter#3 grasp-1] Gripping Sequence implemented and tested

File: robotarm_description/urdf/robotArm.gazebo.xacro (robot description, xacro)
@@ -28,5 +28,5 @@
     <material>Gazebo/Black</material>
     <static>true</static>
-    <turnGravityOff>true</turnGravityOff>
+    <!--turnGravityOff>true</turnGravityOff-->
 </gazebo>
  <gazebo reference="base_link_2">

File: robotarm_description/urdf/robotArm.xacro (robot description, xacro)
@@ -51,9 +51,9 @@
   <property name="left_gripper_len" value="0.08" />
   <property name="left_gripper_width" value="0.01" />
-  <property name="left_gripper_height" value="0.01" />
+  <property name="left_gripper_height" value="0.03" />
   <!-- Right gripper -->
   <property name="right_gripper_len" value="0.08" />
   <property name="right_gripper_width" value="0.01" />
-  <property name="right_gripper_height" value="0.01" />
+  <property name="right_gripper_height" value="0.03" />
   <!-- Right gripper -->
   <property name="grasp_frame_len" value="0.02" />
@@ -84,5 +84,5 @@
       </geometry>
       </collision>>
-      <xacro:inertial_matrix mass="10"/>
+      <xacro:inertial_matrix mass="100"/>
   </link>
   <gazebo reference="bottom_link">
@@ -306,5 +306,5 @@
     <origin xyz="0.0 0 0" />
     <axis xyz="0 1 0" />
-      <limit effort="100" lower="0.03" upper="0" velocity="1.0"/>
+      <limit effort="100" lower="0" upper="0.03" velocity="1.0"/>
       <safety_controller k_position="20"
                          k_velocity="20"
@@ -323,4 +323,10 @@
       <material name="White" />
     </visual>
+    <collision>
+      <origin xyz="0.04 -0.03 0"/>
+      <geometry>
+            <box size="${left_gripper_len} ${left_gripper_width} ${left_gripper_height}" />
+      </geometry>
+    </collision>
   <xacro:inertial_matrix mass="1"/>
   </link>
@@ -347,4 +353,10 @@
       <material name="White" />
     </visual>
+    <collision>
+      <origin xyz="0.04 0.03 0"/>
+      <geometry>
+            <box size="${right_gripper_len} ${right_gripper_width} ${right_gripper_height}" />
+      </geometry>
+    </collision>
   <xacro:inertial_matrix mass="1"/>
   </link>

Commit message: [Iter#3 integrate-1] Combined moveit and grasping node in a single launch file

File: robotarm_description/urdf/robotArm.gazebo.xacro (robot description, xacro)
@@ -82,5 +82,5 @@
 </gazebo>
  <gazebo reference="bottom_link">
-    <static>true</static>
+    <!--static>true</static-->
     <!-- turnGravityOff>true</turnGravityOff -->
 </gazebo>

File: robotarm_description/urdf/robotArm.xacro (robot description, xacro)
@@ -49,9 +49,9 @@
   <property name="gripper_roll_len" value="0.02" />
   <!-- Left gripper -->
-  <property name="left_gripper_len" value="0.08" />
+  <property name="left_gripper_len" value="0.075" />
   <property name="left_gripper_width" value="0.01" />
   <property name="left_gripper_height" value="0.03" />
   <!-- Right gripper -->
-  <property name="right_gripper_len" value="0.08" />
+  <property name="right_gripper_len" value="0.075" />
   <property name="right_gripper_width" value="0.01" />
   <property name="right_gripper_height" value="0.03" />
@@ -83,6 +83,6 @@
          <box size="0.2 0.2 0.02" />
       </geometry>
-      </collision-->
-      <xacro:inertial_matrix mass="90"/>
+      </collision>
+      <xacro:inertial_matrix mass="100"/-->
   </link>
   <gazebo reference="bottom_link">
