Commit message: [Iter#2 simset-5] Camera Setup Successfully. Read for object Detection

File: robotarm_description/urdf/sensors/camera.gazebo.xacro (robot description, xacro)
@@ -9,5 +9,5 @@
       <update_rate>30.0</update_rate>
       <camera name="head">
-        <horizontal_fov>0.95</horizontal_fov>
+        <horizontal_fov>1.3</horizontal_fov>
         <!-- <horizontal_fov>0.95</horizontal_fov> -->
         <image>

File: robotarm_description/urdf/sensors/camera.urdf.xacro (robot description, xacro)
@@ -5,5 +5,5 @@
 <robot name="six_dof_arm" xmlns:xacro="http://www.ros.org/wiki/xacro">
 <joint name="camera_joint" type="fixed">
-    <origin xyz="0 0.2 2" rpy="${M_PI} 0 0"/>
+    <origin xyz="0 0.2 5" rpy="0 ${M_PI/2} 0"/>
     <parent link="base_link"/>
     <child link="camera_link"/>
@@ -12,5 +12,5 @@
    <link name="camera_link">
    <collision>
-   <origin xyz="0 0 0.05" rpy="${-M_PI/2} 0 0"/>
+   <origin xyz="0 0 0" rpy="0 0 0"/>
    <geometry>
    <mesh filename="package://robotarm_description/meshes/camera.STL" />
@@ -18,5 +18,5 @@
    </collision>
    <visual>
-   <origin xyz="0 0 0.05" rpy="${-M_PI/2}  0 0"/>
+   <origin xyz="0 0 0" rpy="${-M_PI} 0 ${-M_PI/2}"/>
    <geometry>
    <mesh filename="package://robotarm_description/meshes/camera.STL" />
@@ -26,5 +26,5 @@
    <inertial>
    <mass value="1e-5" />
-   <origin xyz="0 0 0.05" rpy="${-M_PI/2}  0 0"/>
+   <origin xyz="0 0 0" rpy="0  0 0"/>
    <inertia ixx="1e-6" ixy="0" ixz="0" iyy="1e-6" iyz="0" izz="1e-6" />
    </inertial>
